Commit message: update

File: description/robot_core.xacro (robot description, xacro)
@@ -1,4 +1,33 @@
 <?xml version="1.0"?>
-<robot xmlns:xacro="http://www.ros.org/wiki/xacro"  name="mobile_bot">
-    <link name="base_link"></link>
+<robot xmlns:xacro="http://www.ros.org/wiki/xacro">
+    <material name="white">
+        <color rgba="1 1 1 1" />
+    </material>
+    <material name="orange">
+        <color rgba="1 0.3 0.1 1" />
+    </material>
+    <material name="blue">
+        <color rgba="0.2 0.2 1 1" />
+    </material>
+    <material name="black">
+        <color rgba="0 0 0 1" />
+    </material>
+    <link name="base_link">
+        <!--  -->
+    </link>
+    <!-- joint between base and chassis -->
+    <joint name="base_chassis_joint" type="fixed">
+        <parent link="base_link" />
+        <child link="chassis_link" />
+        <origin xyz="-0.1 0 0" />
+    </joint>
+    <!-- chassis link -->
+    <link name="chassis_link" type="continuous">
+        <visual>
+            <geometry>
+                <box size="0.3 0.3 0.15" />
+                <material name="white" />
+            </geometry>
+        </visual>
+    </link>
 </robot>

Commit message: update

File: description/robot_core.xacro (robot description, xacro)
@@ -27,6 +27,7 @@
             <geometry>
                 <box size="0.3 0.3 0.15" />
-                <material name="white" />
             </geometry>
+            <material name="white" />
+            <origin xyz="0 0 0" />
         </visual>
     </link>

Commit message: 1

File: description/robot_core.xacro (robot description, xacro)
@@ -29,5 +29,5 @@
             </geometry>
             <material name="white" />
-            <origin xyz="0 0 0" />
+            <origin xyz="0.15 0 0.075" />
         </visual>
     </link>

Commit message: 1

File: description/robot_core.xacro (robot description, xacro)
@@ -23,5 +23,5 @@
         <origin xyz="-0.1 0 0" />
     </joint>
-    <link name="chassis_link" type="continuous">
+    <link name="chassis_link">
         <visual>
             <geometry>
@@ -32,3 +32,5 @@
         </visual>
     </link>
+    <!-- left wheel link -->
+    <link name="left_wheel_link"
 </robot>

Commit message: wheels added

File: description/robot_core.xacro (robot description, xacro)
@@ -33,4 +33,32 @@
     </link>
     <!-- left wheel link -->
-    <link name="left_wheel_link"
+    <joint name="base_left_wheel_joint" type="continuous">
+        <parent link="base_link" />
+        <child link="left_wheel_link" />
+        <origin xyz="0 0.175 0" rpy="-${pi/2} 0 0" />
+        <axis xyz="0 0 1" />
+    </joint>
+    <link name="left_wheel_link">
+        <visual>
+            <geometry>
+                <cylinder radius="0.05" length="0.04" />
+            </geometry>
+            <material name="blue" />
+        </visual>
+    </link>
+        <!-- right wheel link -->
+        <joint name="base_right_wheel_joint" type="continuous">
+            <parent link="base_link" />
+            <child link="right_wheel_link" />
+            <origin xyz="0 -0.175 0" rpy="${pi/2} 0 0" />
+            <axis xyz="0 0 -1" />
+        </joint>
+        <link name="right_wheel_link">
+            <visual>
+                <geometry>
+                    <cylinder radius="0.05" length="0.04" />
+                </geometry>
+                <material name="blue" />
+            </visual>
+        </link>
 </robot>

Commit message: 1

File: description/robot_core.xacro (robot description, xacro)
@@ -62,3 +62,17 @@
             </visual>
         </link>
+        <!-- caster wheel link -->
+        <joint name="base_caster_wheel_joint" type="fixed">
+            <parent link="base_link" />
+            <child link="caster_wheel_link" />
+            <origin xyz="0.24 0 0" />
+        </joint>
+        <link name="caster_wheel_link">
+            <visual>
+                <geometry>
+                    <sphere radius="0.05" />
+                </geometry>
+                <material name="blue" />
+            </visual>
+        </link>
 </robot>

Commit message: 1

File: description/robot_core.xacro (robot description, xacro)
@@ -63,6 +63,6 @@
         </link>
         <!-- caster wheel link -->
-        <joint name="base_caster_wheel_joint" type="fixed">
-            <parent link="base_link" />
+        <joint name="chassis_caster_wheel_joint" type="fixed">
+            <parent link="chassis_link" />
             <child link="caster_wheel_link" />
             <origin xyz="0.24 0 0" />
@@ -73,5 +73,5 @@
                     <sphere radius="0.05" />
                 </geometry>
-                <material name="blue" />
+                <material name="black" />
             </visual>
         </link>

Commit message: 1

File: description/robot_core.xacro (robot description, xacro)
@@ -31,4 +31,10 @@
             <origin xyz="0.15 0 0.075" />
         </visual>
+        <collision>
+            <geometry>
+                <box size="0.3 0.3 0.15" />
+            </geometry>
+            <origin xyz="0.15 0 0.075" />
+        </collision>
     </link>
     <!-- left wheel link -->

Commit message: 1

File: description/robot_core.xacro (robot description, xacro)
@@ -52,4 +52,9 @@
             <material name="blue" />
         </visual>
+        <collision>
+            <geometry>
+                <cylinder radius="0.05" length="0.04" />
+            </geometry>
+        </collision>
     </link>
         <!-- right wheel link -->
@@ -67,4 +72,9 @@
                 <material name="blue" />
             </visual>
+            <collision>
+                <geometry>
+                    <cylinder radius="0.05" length="0.04" />
+                </geometry>
+            </collision>
         </link>
         <!-- caster wheel link -->
@@ -81,4 +91,9 @@
                 <material name="black" />
             </visual>
+            <collision>
+                <geometry>
+                    <sphere radius="0.05" />
+                </geometry>
+            </collision>
         </link>
 </robot>

Commit message: 1

File: description/robot_core.xacro (robot description, xacro)
@@ -37,4 +37,7 @@
             <origin xyz="0.15 0 0.075" />
         </collision>
+        <xacro:inertial_box mass="0.5" x="0.3" y="0.3" z="0.15">
+            <origin xyz="0.15 0 0.075" rpy="0 0 0" />
+        </xacro:inertial_box>
     </link>
     <!-- left wheel link -->
@@ -57,4 +60,7 @@
             </geometry>
         </collision>
+        <xacro:inertial_cylinder mass="0.1" length="0.04" radius="0.05">
+            <origin xyz="0 0 0" rpy="0 0 0" />
+        </xacro:inertial_cylinder>
     </link>
         <!-- right wheel link -->
@@ -77,4 +83,7 @@
                 </geometry>
             </collision>
+            <xacro:inertial_cylinder mass="0.1" length="0.04" radius="0.05">
+                <origin xyz="0 0 0" rpy="0 0 0" />
+            </xacro:inertial_cylinder>
         </link>
         <!-- caster wheel link -->
@@ -96,4 +105,7 @@
                 </geometry>
             </collision>
+            <xacro:inertial_sphere mass="0.1" radius="0.05">
+                <origin xyz="0 0 0" rpy="0 0 0" />
+            </xacro:inertial_sphere>
         </link>
 </robot>

Commit message: 1

File: description/robot_core.xacro (robot description, xacro)
@@ -42,4 +42,7 @@
         </xacro:inertial_box>
     </link>
+    <gazebo> reference="chassis_link"
+        <material>Gazebo/White</material>
+    </gazebo>
     <!-- left wheel link -->
     <joint name="base_left_wheel_joint" type="continuous">
@@ -65,4 +68,7 @@
         </xacro:inertial_cylinder>
     </link>
+    <gazebo reference="left_wheel_link">
+        <material>Gazebo/Blue</material>
+    </gazebo>
         <!-- right wheel link -->
         <joint name="base_right_wheel_joint" type="continuous">
@@ -88,4 +94,7 @@
             </xacro:inertial_cylinder>
         </link>
+        <gazebo reference="right_wheel_link">
+            <material>Gazebo/Blue</material>
+        </gazebo>
         <!-- caster wheel link -->
         <joint name="chassis_caster_wheel_joint" type="fixed">
@@ -110,3 +119,6 @@
             </xacro:inertial_sphere>
         </link>
+        <gazebo reference="caster_wheel_link">
+            <material>Gazebo/Black</material>
+        </gazebo>
 </robot>
