Commit message: 1

File: description/lidar.xacro (robot description, xacro)
@@ -4,5 +4,21 @@
         <parent link="chassis_link" />
         <child link="laser_frame" />
-        <origin xyz="0 0 0" rpy="0 0 0" />
+        <origin xyz="0.1 0 0.175" rpy="0 0 0" />
     </joint>
+    <link name="laser_frame">
+        <visual>
+            <geometry>
+                <cylinder radius="0.05" length="0.04" />
+            </geometry>
+            <material name="red" />
+        </visual>
+        <collision>
+            <geometry>
+                <cylinder radius="0.05" length="0.04" />
+            </geometry>
+        </collision>
+        <xacro:inertial_cylinder mass="0.1" length="0.04" radius="0.05">
+            <origin xyz="0 0 0" rpy="0 0 0" />
+        </xacro:inertial_cylinder>
+    </link>
 </robot>

File: description/robot_core.xacro (robot description, xacro)
@@ -13,4 +13,7 @@
     <material name="black">
         <color rgba="0 0 0 1" />
+    </material>
+    <material name="red">
+        <color rgba="1 0 0 1" />
     </material>
     <!-- base link -->

Commit message: modified:   description/lidar.xacro

File: description/lidar.xacro (robot description, xacro)
@@ -22,3 +22,36 @@
         </xacro:inertial_cylinder>
     </link>
+    <gazebo reference="laser_frame">
+        <!-- Color definition in Gazebo -->
+        <material>Gazebo/Red</material>
+        <!-- ray type sensor -->
+        <sensor name="laser" type="ray">
+            <!-- x y z roll pitch yall (relative to the world frame) -->
+            <pose> 0 0 0 0 0 0 </pose>
+            <visualize>true</visualize>
+            <update_rate>10</update_rate>
+            <ray>
+                <scan>
+                    <!-- 2D Lidar so no vertical tag -->
+                    <horizontal>
+                        <samples>360</samples>
+                        <min_angle>-3.14</min_angle>
+                        <max_angle>3.14</max_angle>
+                    </horizontal>
+                </scan>
+                <range>
+                    <min>0.3</min>
+                    <max>12</max>
+                </range>
+            </ray>
+            <!-- laser controller plugin -->
+            <plugin name="laser_controller" filename="libgazebo_ros_ray_sensor.so">
+                <ros>
+                    <argument>~/out:=scan</argument>
+                </ros>
+                <output_type>sensor_msgs/LaserScan</output_type>
+                <frame_name>laser_frame</frame_name>
+            </plugin>
+        </sensor>
+    </gazebo>
 </robot>
