Commit message: modified:   description/depth_camera.xacro

File: description/depth_camera.xacro (robot description, xacro)
@@ -1,28 +1,28 @@
 <?xml version="1.0"?>
 <robot xmlns:xacro="http://www.ros.org/wiki/xacro">
-    <joint name="chassis_camera_joint" type="fixed">
+    <joint name="chassis_depth_camera_joint" type="fixed">
         <parent link="chassis_link" />
-        <child link="camera_link" />
-        <origin xyz="0.305 0 0.08" rpy="0 0 0" />
+        <child link="depth_camera_link" />
+        <origin xyz="0.305 0 0.12" rpy="0 0 0" />
     </joint>
-    <link name="camera_link">
+    <link name="depth_camera_link">
         <visual>
             <geometry>
-                <box size="0.01 0.03 0.03" />
+                <box size="0.01 0.06 0.01" />
             </geometry>
-            <material name="red" />
+            <material name="black" />
         </visual>
     </link>
-    <joint name="chassis_camera_optical_joint" type="fixed">
-        <parent link="camera_link" />
-        <child link="camera_optical_link" />
+    <joint name="chassis_depth_camera_optical_joint" type="fixed">
+        <parent link="depth_camera_link" />
+        <child link="depth_camera_optical_link" />
         <origin xyz="0 0 0" rpy="${-pi/2} 0 ${-pi/2}" />
     </joint>
-    <link name="camera_optical_link"></link>
-    <gazebo reference="camera_link">
+    <link name="depth_camera_optical_link"></link>
+    <gazebo reference="depth_camera_link">
         <!-- Color definition in Gazebo -->
-        <material>Gazebo/Red</material>
+        <material>Gazebo/Black</material>
         <!-- Sensor tag for camera -->
-        <sensor name="camera" type="camera">
+        <sensor name="depth_camera" type="depth">
             <pose> 0 0 0 0 0 0 </pose>
             <visualize>true</visualize>
@@ -45,6 +45,6 @@
             </camera>
             <!-- gazebo camera control plugin -->
-            <plugin name="camera_controller" filename="libgazebo_ros_camera.so">
-                <frame_name>camera_link_optical</frame_name>
+            <plugin name="depth_camera_controller" filename="libgazebo_ros_camera.so">
+                <frame_name>depth_camera_link_optical</frame_name>
             </plugin>
         </sensor>
