Commit message: new file:   config/my_controllers.yaml

File: description/robot.urdf.xacro (robot description, xacro)
@@ -2,8 +2,8 @@
 <robot xmlns:xacro="http://www.ros.org/wiki/xacro"  name="robot">
     <xacro:include filename="robot_core.xacro" />
-    <xacro:include filename="gazebo_control.xacro"/>
+    <!-- <xacro:include filename="gazebo_control.xacro"/> -->
+    <xacro:include filename="ros2_control.xacro"/>
     <xacro:include filename="lidar.xacro"/>
     <xacro:include filename="camera.xacro"/>
     <!-- <xacro:include filename="depth_camera.xacro"/> -->
-    <xacro:include filename="ros2_control.xacro"/>
 </robot>

File: description/ros2_control.xacro (robot description, xacro)
@@ -1,6 +1,36 @@
 <?xml version="1.0"?>
 <robot xmlns:xacro="http://www.ros.org/wiki/xacro">
+    <ros2_control name="GazeboSystem" type="system">
+        <!-- hardware type to be a gazebo system -->
+        <hardware>
+            <plugin>gazebo_ros2_control/GazeboSystem</plugin>
+        </hardware>
+        <joint name="base_left_wheel_joint">
+            <!-- command interfaces -->
+            <command_interface name="velocity">
+                <param name="min">-10</param>
+                <param name="max">10</param>
+            </command_interface>
+            <!-- state interfaces -->
+            <state_interface name="velocity" />
+            <state_interface name="position" />
+        </joint>
+        <joint name="base_right_wheel_joint">
+            <!-- command interfaces -->
+            <command_interface name="velocity">
+                <param name="min">-10</param>
+                <param name="max">10</param>
+            </command_interface>
+            <!-- state interfaces -->
+            <state_interface name="velocity" />
+            <state_interface name="position" />
+        </joint>
+    </ros2_control>
     <gazebo>
-        <plugin name="diff_drive" filename="libgazebo_ros_diff_drive.so">
+        <plugin name="diff_drive" filename="libgazebo.ros_diff_drive.so">
+        </plugin>
+    </gazebo>
+    <gazebo>
+        <plugin name="gazebo_ros2_control" filename="libgazebo_ros2_control.so">
             <!-- Wheel Information -->
             <left_joint>base_left_wheel_joint</left_joint>
